Commit message: 双船模型

File: build/vrx/wamv_description/urdf/wamv_base.urdf (robot description, URDF)
Before this commit: robot wam-v, 2 links, 1 joints
Links:
- link dummy_link: geometry collision box size=0.65 0.2 0.1; collision box size=0.65 0.2 0.1

File: build/vrx/wamv_gazebo/urdf/wamv_gazebo.urdf (robot description, URDF)
Before this commit: robot WAM-V, 8 links, 7 joints
Links:
- link dummy_link: geometry collision box size=0.65 0.2 0.1; collision box size=0.65 0.2 0.1
- link left_battery_link: geometry collision box size=.6 .4 .31; visual mesh filename=package://vrx_gazebo/models/battery/mesh/battery.dae
- link left_engine_link: geometry collision box size=0.12 0.15 0.12; collision box size=0.2 0.15 0.83
- link left_propeller_link: geometry collision cylinder length=0.18 radius=0.24; visual mesh filename=package://wamv_description/models/propeller/mesh/propeller.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
- link right_battery_link: geometry collision box size=.6 .4 .31; visual mesh filename=package://vrx_gazebo/models/battery/mesh/battery.dae
- link right_engine_link: geometry collision box size=0.12 0.15 0.12; collision box size=0.2 0.15 0.83
- link right_propeller_link: geometry collision cylinder length=0.18 radius=0.24; visual mesh filename=package://wamv_description/models/propeller/mesh/propeller.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

File: src/vrx/vrx_gazebo/worlds/dock.world.xacro (robot description, xacro)
@@ -8,39 +8,20 @@
     <xacro:include filename="$(find wave_gazebo)/world_models/ocean_waves/model.xacro"/>
     <xacro:ocean_waves/>
+    <!--wind for the wamv-->
+    <xacro:include filename="$(find vrx_gazebo)/worlds/xacros/usv_wind_plugin.xacro"/>
+    <xacro:usv_wind_gazebo>
+      <wind_objs>
+        <wind_obj>
+          <name>wamv</name>
+          <link_name>base_link</link_name>
+          <coeff_vector>.5 .5 .33</coeff_vector>
+        </wind_obj>
+      </wind_objs>
+    </xacro:usv_wind_gazebo>
     <!-- The 2018 dock with the two placards -->
     <include>
-      <uri>model://dock_2018</uri>
-      <pose>60 -2.75 0 0 0 0</pose>
+      <uri>model://dock_2018_dynamic</uri>
+      <pose>130 97 0 0 0 0</pose>
     </include>
-    <!-- Uncomment to visualize the bay #1 activation zone -->
-    <!-- <model name="activation_placard1">
-      <static>true</static>
-      <link name="link">
-        <visual name="visual">
-          <pose>72.75 0 0 0 0 0</pose>
-          <geometry>
-            <box>
-              <size>1.5 4 2</size>
-            </box>
-          </geometry>
-          <transparency>0.8</transparency>
-        </visual>
-      </link>
-    </model> -->
-    <!-- Uncomment to visualize the bay #2 activation zone -->
-    <!-- <model name="activation_placard2">
-      <static>true</static>
-      <link name="link">
-        <visual name="visual">
-          <pose>61.75 0 0 0 0 0</pose>
-          <geometry>
-            <box>
-              <size>1.5 4 2</size>
-            </box>
-          </geometry>
-          <transparency>0.8</transparency>
-        </visual>
-      </link>
-    </model> -->
     <!-- The scoring plugin -->
     <plugin name="scan_dock_scoring_plugin"
@@ -48,7 +29,7 @@
       <!-- Parameters for scoring_plugin -->
       <vehicle>wamv</vehicle>
-      <task_name>scan_dock</task_name>
-      <initial_state_duration>3</initial_state_duration>
-      <ready_state_duration>3</ready_state_duration>
+      <task_name>scan</task_name>
+      <initial_state_duration>10</initial_state_duration>
+      <ready_state_duration>10</ready_state_duration>
       <running_state_duration>300</running_state_duration>
       <release_joints>
@@ -62,4 +43,5 @@
       <!-- Color sequence checker -->
       <robot_namespace>vrx</robot_namespace>
+      <enable_color_checker>False</enable_color_checker>
       <color_sequence_service>scan_dock/color_sequence</color_sequence_service>
       <color_1>red</color_1>
@@ -70,5 +52,6 @@
         <bay>
           <name>bay1</name>
-          <activation_topic>/vrx/dock_2018/bay_1/contain</activation_topic>
+          <internal_activation_topic>/vrx/dock_2018/bay_1_internal/contain</internal_activation_topic>
+          <external_activation_topic>/vrx/dock_2018/bay_1_external/contain</external_activation_topic>
           <symbol_topic>/vrx/dock_2018_placard1/symbol</symbol_topic>
           <min_dock_time>10.0</min_dock_time>
@@ -78,18 +61,19 @@
         <bay>
           <name>bay2</name>
-          <activation_topic>/vrx/dock_2018/bay_2/contain</activation_topic>
+          <internal_activation_topic>/vrx/dock_2018/bay_2_internal/contain</internal_activation_topic>
+          <external_activation_topic>/vrx/dock_2018/bay_2_external/contain</external_activation_topic>
           <symbol_topic>/vrx/dock_2018_placard2/symbol</symbol_topic>
           <min_dock_time>10.0</min_dock_time>
+          <!-- Set this bay as the intended docking bay -->
           <dock_allowed>true</dock_allowed>
-          <announce_symbol>red_cross</announce_symbol>
+          <!-- Specify the visual symbol - should be same as announced -->
           <symbol>red_cross</symbol>
         </bay>
       </bays>
-      <placard_color_shape>red_cross</placard_color_shape>
     </plugin>
     <!-- Triggers a message when the vehicle enters and exits the bay #1 -->
     <plugin name="vehicle_docked_bay1" filename="libContainPlugin.so">
       <entity>wamv::base_link</entity>
-      <namespace>vrx/dock_2018/bay_1</namespace>
+      <namespace>vrx/dock_2018/bay_1_internal</namespace>
       <pose frame="robotx_dock_2018::dock_2018_placard1::placard::link">0 -5 -1.5 0 0 0</pose>
       <geometry>
@@ -99,8 +83,19 @@
       </geometry>
     </plugin>
+    <!-- Triggers a message when the vehicle enters and exits the bay #1 -->
+    <plugin name="vehicle_docked_bay1_exterior" filename="libContainPlugin.so">
+      <entity>wamv::base_link</entity>
+      <namespace>vrx/dock_2018/bay_1_external</namespace>
+      <pose frame="robotx_dock_2018::dock_2018_placard1::placard::link">0 -10 -1.5 0 0 0</pose>
+      <geometry>
+        <box>
+          <size>8 1.5 2</size>
+        </box>
+      </geometry>
+    </plugin>
     <!-- Triggers a message when the vehicle enters and exits the bay #2 -->
     <plugin name="vehicle_docked_bay2" filename="libContainPlugin.so">
       <entity>wamv::base_link</entity>
-      <namespace>vrx/dock_2018/bay_2</namespace>
+      <namespace>vrx/dock_2018/bay_2_internal</namespace>
       <pose frame="robotx_dock_2018::dock_2018_placard2::placard::link">0 5 -1.5 0 0 0</pose>
       <geometry>
@@ -110,4 +105,15 @@
       </geometry>
     </plugin>
+    <!-- Triggers a message when the vehicle enters and exits the bay #1 -->
+    <plugin name="vehicle_docked_bay2_exterior" filename="libContainPlugin.so">
+      <entity>wamv::base_link</entity>
+      <namespace>vrx/dock_2018/bay_2_external</namespace>
+      <pose frame="robotx_dock_2018::dock_2018_placard1::placard::link">0 10 -1.5 0 0 0</pose>
+      <geometry>
+        <box>
+          <size>8 1.5 2</size>
+        </box>
+      </geometry>
+    </plugin>
   </world>
 </sdf>

File: src/vrx/vrx_gazebo/worlds/example_course.world.xacro (robot description, xacro)
@@ -23,10 +23,10 @@
     <include>
       <uri>model://dock_2016</uri>
-      <pose>75 22 0 0 0 -2.78</pose>
+      <pose>75 22 0.0 0 0 -2.78</pose>
     </include>
     <!-- The 2018 dock with the two placards -->
     <include>
       <uri>model://dock_2018</uri>
-      <pose>-2 -18 0 0 0 0.2</pose>
+      <pose>-2 -18 0.0 0 0 0.2</pose>
     </include>
     <xacro:include filename="$(find vrx_gazebo)/worlds/xacros/usv_wind_plugin.xacro"/>

File: src/vrx/vrx_gazebo/worlds/perception_task.world.xacro (robot description, xacro)
@@ -34,5 +34,5 @@
       <running_state_duration>300</running_state_duration>
       <!-- Parameters for PopulationPlugin -->
-      <loop_forever>false</loop_forever>
+      <loop_forever>true</loop_forever>
       <frame>wamv</frame>
       <!-- Pose of each object is expressed relative to the body frame
@@ -41,19 +41,19 @@
       <object_sequence>
         <object>
-          <time>5.0</time>
-          <type>red</type>
-          <name>red_mark</name>
-            <pose>8 0 1 0 0 0</pose>
+          <time>5</time>
+          <type>surmark950410</type>
+          <name>red_0</name>
+          <pose>8 0 1 0 0 0</pose>
         </object>
         <object>
-          <time>10.0</time>
-          <type>green</type>
-          <name>green_mark</name>
+          <time>5</time>
+          <type>surmark950400</type>
+          <name>green_0</name>
           <pose>8 2 1 0 0 0</pose>
         </object>
         <object>
           <time>15.0</time>
-          <type>black</type>
-          <name>black_totem</name>
+          <type>black_totem</type>
+          <name>black_0</name>
           <pose>8 -2 1 0 0 0</pose>
         </object>

File: src/vrx/vrx_gazebo/worlds/scan_and_dock.world.xacro (robot description, xacro)
@@ -7,5 +7,16 @@
     <!--Waves-->
     <xacro:include filename="$(find wave_gazebo)/world_models/ocean_waves/model.xacro"/>
-    <xacro:ocean_waves/>>
+    <xacro:ocean_waves/>
+    <!--wind for the wamv-->
+    <xacro:include filename="$(find vrx_gazebo)/worlds/xacros/usv_wind_plugin.xacro"/>
+    <xacro:usv_wind_gazebo>
+      <wind_objs>
+        <wind_obj>
+          <name>wamv</name>
+          <link_name>base_link</link_name>
+          <coeff_vector>.5 .5 .33</coeff_vector>
+        </wind_obj>
+      </wind_objs>
+    </xacro:usv_wind_gazebo>
     <!-- The light buoy -->
     <include>
@@ -53,5 +64,5 @@
       <!-- Parameters for scoring_plugin -->
       <vehicle>wamv</vehicle>
-      <task_name>scan_dock</task_name>
+      <task_name>scan_and_dock</task_name>
       <initial_state_duration>3</initial_state_duration>
       <ready_state_duration>3</ready_state_duration>
@@ -75,5 +86,6 @@
         <bay>
           <name>bay1</name>
-          <activation_topic>/vrx/dock_2018/bay_1/contain</activation_topic>
+          <internal_activation_topic>/vrx/dock_2018/bay_1/contain</internal_activation_topic>
+          <external_activation_topic>/vrx/dock_2018/bay_1_exterior/contain</external_activation_topic>
           <symbol_topic>/vrx/dock_2018_placard1/symbol</symbol_topic>
 	        <min_dock_time>10.0</min_dock_time>
@@ -83,5 +95,6 @@
         <bay>
           <name>bay2</name>
-          <activation_topic>/vrx/dock_2018/bay_2/contain</activation_topic>
+          <internal_activation_topic>/vrx/dock_2018/bay_2/contain</internal_activation_topic>
+          <external_activation_topic>/vrx/dock_2018/bay_2_exterior/contain</external_activation_topic>
           <symbol_topic>/vrx/dock_2018_placard2/symbol</symbol_topic>
           <min_dock_time>10.0</min_dock_time>

File: src/vrx/vrx_gazebo/worlds/stationkeeping_task.world.xacro (robot description, xacro)
@@ -8,4 +8,15 @@
     <xacro:include filename="$(find wave_gazebo)/world_models/ocean_waves/model.xacro"/>
     <xacro:ocean_waves/>
+    <!--wind for the wamv-->
+    <xacro:include filename="$(find vrx_gazebo)/worlds/xacros/usv_wind_plugin.xacro"/>
+    <xacro:usv_wind_gazebo>
+      <wind_objs>
+        <wind_obj>
+          <name>wamv</name>
+          <link_name>base_link</link_name>
+          <coeff_vector>.5 .5 .33</coeff_vector>
+        </wind_obj>
+      </wind_objs>
+    </xacro:usv_wind_gazebo>
   <plugin name="stationkeeping_scoring_plugin"
           filename="libstationkeeping_scoring_plugin.so">
@@ -25,4 +36,8 @@
         </joint>
       </release_joints>
+      <markers>
+        <scaling>0.2 0.2 2.0</scaling>
+        <height>0.5</height>
+      </markers>
     </plugin>
   </world>

File: src/vrx/vrx_gazebo/worlds/wayfinding_task.world.xacro (robot description, xacro)
@@ -8,4 +8,15 @@
     <xacro:include filename="$(find wave_gazebo)/world_models/ocean_waves/model.xacro"/>
     <xacro:ocean_waves/>
+    <!--wind for the wamv-->
+    <xacro:include filename="$(find vrx_gazebo)/worlds/xacros/usv_wind_plugin.xacro"/>
+    <xacro:usv_wind_gazebo>
+      <wind_objs>
+        <wind_obj>
+          <name>wamv</name>
+          <link_name>base_link</link_name>
+          <coeff_vector>.5 .5 .33</coeff_vector>
+        </wind_obj>
+      </wind_objs>
+    </xacro:usv_wind_gazebo>
     <plugin name="wayfinding_scoring_plugin"
             filename="libwayfinding_scoring_plugin.so">
@@ -38,4 +49,8 @@
         </joint>
       </release_joints>
+      <markers>
+        <scaling>0.2 0.2 2.0</scaling>
+        <height>0.5</height>
+      </markers>
     </plugin>
   </world>

File: src/vrx/vrx_gazebo/worlds/xacros/dock.xacro (robot description, xacro)
@@ -2,5 +2,13 @@
 <!-- World containing sandisland model and some course challenges -->
 <world xmlns:xacro="http://ros.org/wiki/xacro">
-  <xacro:macro name="dock" params="uri:=dock_2018 x:=60 y:=-2.75 z:=0 R:=0 P:=0 Y:=0">
+  <xacro:macro name="dock" params="model_name:=robotx_dock_2018
+    uri:=dock_2018 x:=60 y:=-2.75 z:=0
+    R:=0 P:=0 Y:=0 bay1_allowed:=false bay1_symbol:=red_circle
+    bay2_allowed:=true bay2_symbol:=blue_cross
+    light_buoy_present:=false
+    color_1:=red color_2:=green color_3:=blue
+    lb_x:=90 lb_y:=70 lb_z:=0 lb_R:=0 lb_P:=0 lb_Y:=0
+    enable_color_checker:=false
+		task_name:=dock">
     <!-- The 2018 dock with the two placards -->
     <include>
@@ -8,4 +16,11 @@
       <pose>${x} ${y} ${z} ${R} ${P} ${Y}</pose>
     </include>
+    <!-- Add a ligth buoy if doing Scan and Dock -->
+    <xacro:if value="${light_buoy_present}">
+      <include>
+        <uri>model://robotx_light_buoy</uri>
+        <pose>${lb_x} ${lb_y} ${lb_z} ${lb_R} ${lb_P} ${lb_Y}</pose>
+      </include>
+    </xacro:if>
     <!-- The scoring plugin -->
     <plugin name="scan_dock_scoring_plugin"
@@ -13,7 +28,7 @@
       <!-- Parameters for scoring_plugin -->
       <vehicle>wamv</vehicle>
-      <task_name>scan_dock</task_name>
-      <initial_state_duration>3</initial_state_duration>
-      <ready_state_duration>3</ready_state_duration>
+      <task_name>${task_name}</task_name>
+      <initial_state_duration>10</initial_state_duration>
+      <ready_state_duration>10</ready_state_duration>
       <running_state_duration>300</running_state_duration>
       <release_joints>
@@ -26,36 +41,37 @@
       </release_joints>
       <!-- Color sequence checker -->
+      <enable_color_checker>${enable_color_checker}</enable_color_checker>
       <robot_namespace>vrx</robot_namespace>
       <color_sequence_service>scan_dock/color_sequence</color_sequence_service>
-      <color_1>red</color_1>
-      <color_2>green</color_2>
-      <color_3>blue</color_3>
+      <color_1>${color_1}</color_1>
+      <color_2>${color_2}</color_2>
+      <color_3>${color_3}</color_3>
       <!-- Dock checkers -->
       <bays>
         <bay>
           <name>bay1</name>
-          <activation_topic>/vrx/dock_2018/bay_1/contain</activation_topic>
+          <internal_activation_topic>/vrx/dock_2018/bay_1_internal/contain</internal_activation_topic>
+          <external_activation_topic>/vrx/dock_2018/bay_1_external/contain</external_activation_topic>
           <symbol_topic>/vrx/dock_2018_placard1/symbol</symbol_topic>
           <min_dock_time>10.0</min_dock_time>
-          <dock_allowed>false</dock_allowed>
-          <symbol>red_circle</symbol>
+          <dock_allowed>${bay1_allowed}</dock_allowed>
+          <symbol>${bay1_symbol}</symbol>
         </bay>
         <bay>
           <name>bay2</name>
-          <activation_topic>/vrx/dock_2018/bay_2/contain</activation_topic>
+          <internal_activation_topic>/vrx/dock_2018/bay_2_internal/contain</internal_activation_topic>
+          <external_activation_topic>/vrx/dock_2018/bay_2_external/contain</external_activation_topic>
           <symbol_topic>/vrx/dock_2018_placard2/symbol</symbol_topic>
           <min_dock_time>10.0</min_dock_time>
-          <dock_allowed>true</dock_allowed>
-          <announce_symbol>red_cross</announce_symbol>
-          <symbol>red_cross</symbol>
+          <dock_allowed>${bay2_allowed}</dock_allowed>
+          <symbol>${bay2_symbol}</symbol>
         </bay>
       </bays>
-      <placard_color_shape>red_triangle</placard_color_shape>
     </plugin>
     <!-- Triggers a message when the vehicle enters and exits the bay #1 -->
     <plugin name="vehicle_docked_bay1" filename="libContainPlugin.so">
       <entity>wamv::base_link</entity>
-      <namespace>vrx/dock_2018/bay_1</namespace>
-      <pose frame="robotx_dock_2018::dock_2018_placard1::placard::link">0 -5 -1.5 0 0 0</pose>
+      <namespace>vrx/dock_2018/bay_1_internal</namespace>
+      <pose frame="${model_name}::dock_2018_placard1::placard::link">0 -5 -1.5 0 0 0</pose>
       <geometry>
         <box>
@@ -64,9 +80,20 @@
       </geometry>
     </plugin>
+    <!-- Triggers a message when the vehicle enters and exits the bay #1 -->
+    <plugin name="vehicle_docked_bay1_exterior" filename="libContainPlugin.so">
+      <entity>wamv::base_link</entity>
+      <namespace>vrx/dock_2018/bay_1_external</namespace>
+      <pose frame="${model_name}::dock_2018_placard1::placard::link">0 -10 -1.5 0 0 0</pose>
+      <geometry>
+        <box>
+          <size>8 1.5 2</size>
+        </box>
+      </geometry>
+    </plugin>
     <!-- Triggers a message when the vehicle enters and exits the bay #2 -->
     <plugin name="vehicle_docked_bay2" filename="libContainPlugin.so">
       <entity>wamv::base_link</entity>
-      <namespace>vrx/dock_2018/bay_2</namespace>
-      <pose frame="robotx_dock_2018::dock_2018_placard2::placard::link">0 5 -1.5 0 0 0</pose>
+      <namespace>vrx/dock_2018/bay_2_internal</namespace>
+      <pose frame="${model_name}::dock_2018_placard2::placard::link">0 5 -1.5 0 0 0</pose>
       <geometry>
         <box>
@@ -75,4 +102,15 @@
       </geometry>
     </plugin>
+    <!-- Triggers a message when the vehicle enters and exits the bay #1 -->
+    <plugin name="vehicle_docked_bay2_exterior" filename="libContainPlugin.so">
+      <entity>wamv::base_link</entity>
+      <namespace>vrx/dock_2018/bay_2_external</namespace>
+      <pose frame="${model_name}::dock_2018_placard1::placard::link">0 10 -1.5 0 0 0</pose>
+      <geometry>
+        <box>
+          <size>8 1.5 2</size>
+        </box>
+      </geometry>
+    </plugin>
   </xacro:macro>
 </world>

File: src/vrx/vrx_gazebo/worlds/xacros/include_all_xacros.xacro (robot description, xacro)
@@ -6,4 +6,9 @@
     <xacro:include filename="$(find vrx_gazebo)/worlds/xacros/scene.xacro" />
     <xacro:include filename="$(find vrx_gazebo)/worlds/xacros/nav_challenge.xacro" />
+    <!-- <xacro:include filename="$(find vrx_gazebo)/worlds/xacros/light_buoy.xacro" />
+    <xacro:include filename="$(find vrx_gazebo)/worlds/xacros/qualifying_pinger_transit_2016.xacro" />
+    <xacro:include filename="$(find vrx_gazebo)/worlds/xacros/dock_2016.xacro" />
+    <xacro:include filename="$(find vrx_gazebo)/worlds/xacros/dock_2018.xacro" />
+    <xacro:include filename="$(find vrx_gazebo)/worlds/xacros/scene_macro.xacro" /> -->
     <xacro:include filename="$(find vrx_gazebo)/worlds/xacros/usv_wind_plugin.xacro" />
     <xacro:include filename="$(find wave_gazebo)/world_models/ocean_waves/model.xacro"/>
@@ -13,4 +18,5 @@
     <xacro:include filename="$(find vrx_gazebo)/worlds/xacros/scan_and_dock.xacro" />
     <xacro:include filename="$(find vrx_gazebo)/worlds/xacros/wayfinding.xacro" />
+    <xacro:include filename="$(find vrx_gazebo)/worlds/xacros/insert_model.xacro" />
   </xacro:macro>
 </world>

File: src/vrx/vrx_gazebo/worlds/xacros/scan_and_dock.xacro (robot description, xacro)
@@ -19,6 +19,6 @@
       <vehicle>wamv</vehicle>
       <task_name>scan_dock</task_name>
-      <initial_state_duration>3</initial_state_duration>
-      <ready_state_duration>3</ready_state_duration>
+      <initial_state_duration>10</initial_state_duration>
+      <ready_state_duration>10</ready_state_duration>
       <running_state_duration>300</running_state_duration>
       <release_joints>
@@ -40,5 +40,6 @@
         <bay>
           <name>bay1</name>
-          <activation_topic>/vrx/dock_2018/bay_1/contain</activation_topic>
+          <internal_activation_topic>/vrx/dock_2018/bay_1/contain</internal_activation_topic>
+          <external_activation_topic>/vrx/dock_2018/bay_1_exterior/contain</external_activation_topic>
           <symbol_topic>/vrx/dock_2018_placard1/symbol</symbol_topic>
           <min_dock_time>10.0</min_dock_time>
@@ -48,13 +49,12 @@
         <bay>
           <name>bay2</name>
-          <activation_topic>/vrx/dock_2018/bay_2/contain</activation_topic>
+          <internal_activation_topic>/vrx/dock_2018/bay_2/contain</internal_activation_topic>
+          <external_activation_topic>/vrx/dock_2018/bay_2_exterior/contain</external_activation_topic>
           <symbol_topic>/vrx/dock_2018_placard2/symbol</symbol_topic>
           <min_dock_time>10.0</min_dock_time>
           <dock_allowed>true</dock_allowed>
-          <announce_symbol>red_cross</announce_symbol>
           <symbol>red_cross</symbol>
         </bay>
       </bays>
-      <placard_color_shape>red_cross</placard_color_shape>
     </plugin>
   </xacro:macro>

File: src/vrx/wamv_gazebo/urdf/sensors/wamv_3d_lidar.xacro (robot description, xacro)
@@ -39,5 +39,5 @@
         <origin xyz="0 0 -0.035" rpy="0 0 0"/>
         <geometry>
-          <mesh filename="model://3d_lidar/mesh/3d_lidar.dae"/>
+          <mesh filename="package://vrx_gazebo/models/3d_lidar/mesh/3d_lidar.dae"/>
         </geometry>
       </visual>
@@ -94,5 +94,5 @@
         <origin xyz="-0.038 0 -0.003" rpy="${radians(-60)} 0 ${-pi/2}"/>
         <geometry>
-          <mesh filename="model://sensor_post/mesh/sensor_post_arm.dae"/>
+          <mesh filename="package://vrx_gazebo/models/sensor_post/mesh/sensor_post_arm.dae"/>
         </geometry>
       </visual>
@@ -164,6 +164,6 @@
         </ray>
         <plugin name="${name}_plugin" filename="libgazebo_ros_velodyne_gpu_laser.so">
-          <topicName>${name}/points</topicName>
-          <frameName>${name}_link</frameName>
+          <topicName>${namespace}/${sensor_namespace}lidars/${name}/points</topicName>
+          <frameName>${namespace}/${name}_link</frameName>
           <min_intensity>0</min_intensity>
         </plugin>
