Commit message: 双船模型

File: src/vrx/wamv_gazebo/urdf/sensors/wamv_camera.xacro (robot description, xacro)
@@ -12,5 +12,5 @@
         <origin xyz="-0.033 0 0" rpy="0 0 ${pi/2}"/>
         <geometry>
-          <mesh filename="model://mono_camera/mesh/mono_camera.dae"/>
+          <mesh filename="package://vrx_gazebo/models/mono_camera/mesh/mono_camera.dae"/>
         </geometry>
       </visual>
@@ -38,4 +38,8 @@
           iyz="0"/>
       </inertial>
+    </link>
+    <!-- Define a link for the optical frame.  This will match the sensor frame and
+         be oriented in the camera convention. -->
+    <link name="${name}_link_optical">
     </link>
     <!-- Define post length and mass based on desired z position of sensor -->
@@ -75,5 +79,5 @@
         <origin xyz="-0.038 0 -0.003" rpy="${radians(-60)} 0 ${-pi/2}"/>
         <geometry>
-          <mesh filename="model://sensor_post/mesh/sensor_post_arm.dae"/>
+          <mesh filename="package://vrx_gazebo/models/sensor_post/mesh/sensor_post_arm.dae"/>
         </geometry>
       </visual>
@@ -116,4 +120,11 @@
       <child link="${name}_link" />
     </joint>
+    <!-- Camera to optical frame joint.  This is oriented to convert between ENU
+         and camera conventions -->
+    <joint name="${name}_to_${name}_link_optical_joint" type="fixed">
+      <origin xyz="0 0 0" rpy="${-pi/2} 0 ${-pi/2}" />
+      <parent link="${name}_link" />
+      <child link="${name}_link_optical" />
+    </joint>
     <!-- Gazebo camera setup -->
     <gazebo reference="${name}_link">
@@ -143,8 +154,8 @@
           <alwaysOn>true</alwaysOn>
           <updateRate>0.0</updateRate>
-          <cameraName>${name}</cameraName>
+          <cameraName>${namespace}/${sensor_namespace}${camera_namespace}${name}</cameraName>
           <imageTopicName>image_raw</imageTopicName>
           <cameraInfoTopicName>camera_info</cameraInfoTopicName>
-          <frameName>${name}_link_optical</frameName>
+          <frameName>${namespace}/${name}_link_optical</frameName>
           <hackBaseline>0.07</hackBaseline>
           <distortionK1>0.0</distortionK1>

File: src/vrx/wamv_gazebo/urdf/sensors/wamv_gps.xacro (robot description, xacro)
@@ -5,5 +5,5 @@
       <visual name="${name}_visual">
         <geometry>
-          <mesh filename="package://wamv_gazebo/mesh/gps.dae"/>
+          <mesh filename="package://wamv_gazebo/models/gps/mesh/gps.dae"/>
         </geometry>
       </visual>
@@ -25,5 +25,7 @@
       </inertial>
     </link>
-    <joint name="${name}_joint" type="fixed">
+    <joint name="${name}_joint" type="revolute">
+      <axis xyz="0 0 1"/>
+      <limit effort="1000.0" lower="0.0" upper="0" velocity="0"/>
       <origin xyz="${x} ${y} ${z}" rpy="${R} ${P} ${Y}" />
       <parent link="base_link" />
@@ -35,6 +37,7 @@
         <alwaysOn>true</alwaysOn>
         <bodyName>${name}_link</bodyName>
-        <frameId>${name}_link</frameId>
-        <topicName>gps/fix</topicName>
+        <!-- Manually prepend namespace to tf frame. -->
+        <frameId>${namespace}/${name}_link</frameId>
+        <topicName>${namespace}/${sensor_namespace}gps/gps/fix</topicName>
         <!-- Note that the hector_gazebo_ros_gps plugin uses NWU coordinates
              for reporting velocities.  This may cause problems if localization
@@ -42,9 +45,9 @@
              See Issue #64 in VRX project for details
              https://bitbucket.org/osrf/vrx/issues/64 -->
-        <velocityTopicName>gps/fix_velocity</velocityTopicName>
+        <velocityTopicName>${namespace}/${sensor_namespace}gps/gps/fix_velocity</velocityTopicName>
         <!-- Location of origin of Gazebo Sand Island map -->
         <referenceLatitude>21.30996</referenceLatitude>
         <referenceLongitude>-157.8901</referenceLongitude>
-        <referenceAltitude>${z}</referenceAltitude>
+        <referenceAltitude>0</referenceAltitude>
         <referenceHeading>90</referenceHeading>
         <offset>0.0 0.0 0.0</offset>

File: src/vrx/wamv_gazebo/urdf/sensors/wamv_imu.xacro (robot description, xacro)
@@ -11,6 +11,12 @@
         </material>
       </visual>
+      <inertial>
+        <mass value="0.1"/>
+        <inertia ixx="0.000083" ixy="0.0" ixz="0.0" iyy="0.000083" iyz="0.0" izz="0.0125"/>
+      </inertial>
     </link>
-    <joint name="${name}_joint" type="fixed">
+    <joint name="${name}_joint" type="revolute">
+      <axis xyz="0 0 1"/>
+      <limit effort="1000.0" lower="0.0" upper="0" velocity="0"/>
       <origin xyz="${x} ${y} ${z}" rpy="${R} ${P} ${Y}"/>
       <parent link="base_link"/>
@@ -21,7 +27,8 @@
         <updateRate>15.0</updateRate>
         <bodyName>${name}_link</bodyName>
-        <topicName>imu/data</topicName>
-        <serviceName>imu_service</serviceName>
-        <frameId>${name}_link</frameId>
+        <topicName>${namespace}/${sensor_namespace}imu/imu/data</topicName>
+        <serviceName>${namespace}/${sensor_namespace}imu_service</serviceName>
+        <!-- Manually prepend namespace to tf frame. -->
+        <frameId>${namespace}/${name}_link</frameId>
         <alwaysOn>true</alwaysOn>
         <accelOffset>0.0 0.0 0.0</accelOffset>

File: src/vrx/wamv_gazebo/urdf/sensors/wamv_p3d.xacro (robot description, xacro)
@@ -7,5 +7,5 @@
         <frameName>map</frameName>
         <updateRate>10.0</updateRate>
-        <topicName>${name}</topicName>
+        <topicName>${namespace}/${sensor_namespace}position/${name}</topicName>
         <xyzOffset>0 0 0</xyzOffset>
         <rpyOffset>0 0 0</rpyOffset>

File: src/vrx/wamv_gazebo/urdf/sensors/wamv_planar_lidar.xacro (robot description, xacro)
@@ -39,5 +39,5 @@
         </ray>
         <plugin name="multibeam_simulator" filename="libgazebo_ros_gpu_laser.so">
-          <topicName>${name}/scan</topicName>
+          <topicName>${namespace}/${sensor_namespace}lidars/${name}/scan</topicName>
           <frameName>${name}_link</frameName>
         </plugin>

File: src/vrx/wamv_gazebo/urdf/wamv_gazebo.urdf.xacro (robot description, xacro)
@@ -11,4 +11,17 @@
   <xacro:arg name="ground_truth_enabled" default="false" />
   <xacro:arg name="vrx_sensors_enabled" default="false" />
+  <xacro:arg name="pinger_enabled" default="false" />
+  <xacro:arg name="thruster_namespace" default="thrusters/"/>
+  <xacro:arg name="camera_namespace" default="cameras/"/>
+  <xacro:arg name="sensor_namespace" default="sensors/"/>
+  <xacro:arg name="pinger_namespace" default="pingers/"/>
+  <!-- Note: this is only used for some sensors that do not correctly use the
+  robotNamespace parameter -->
+  <xacro:arg name="namespace" default="wamv"/>
+  <xacro:property name="thruster_namespace" value="$(arg thruster_namespace)" scope="global" />
+  <xacro:property name="camera_namespace" value="$(arg camera_namespace)" scope="global" />
+  <xacro:property name="sensor_namespace" value="$(arg sensor_namespace)" scope="global" />
+  <xacro:property name="pinger_namespace" value="$(arg pinger_namespace)" scope="global" />
+  <xacro:property name="namespace" value="$(arg namespace)" scope="global" />
   <!-- Sensor yaml file -->
   <xacro:arg name="yaml_sensor_generation" default="false"/>
@@ -102,4 +115,8 @@
       <xacro:wamv_p3d name="p3d_wamv"/>
     </xacro:if>
+    <!-- Add pinger -->
+    <xacro:if value="$(arg pinger_enabled)">
+      <xacro:wamv_pinger name="pinger" position="1.0 0 -1.0" />
+    </xacro:if>
     <!-- ==== VRX sensor configuration ==== -->
     <xacro:if value="$(arg vrx_sensors_enabled)">
@@ -118,4 +135,6 @@
       <!-- Add 3D LIDAR -->
       <xacro:lidar name="lidar_wamv" type="16_beam"/>
+      <!-- Add pinger -->
+      <xacro:wamv_pinger name="pinger" position="1.0 0 -1.0" />
     </xacro:if>
   </xacro:unless>
